Commit message: Initial commit swerve_bringup

File: urdf/swerve_base.urdf (robot description, URDF)
Before this commit: robot agv_base, 12 links, 11 joints
Links:
- added link v30e_link; visual box size=0.09 0.07 0.025
- link wheel_front_left_link: geometry collision cylinder length=0.040 radius=0.040; visual sphere radius=0.0414
- link wheel_front_right_link: geometry collision cylinder length=0.040 radius=0.040; visual sphere radius=0.0414
- link wheel_rear_left_link: geometry collision cylinder length=0.040 radius=0.040; visual sphere radius=0.043
- link wheel_rear_right_link: geometry collision cylinder length=0.040 radius=0.040; visual sphere radius=0.043
Joints:
- added joint base_v30e_joint: type fixed, parent base_link, child v30e_link, origin xyz=0 0 -0.145 rpy=0 0 0
- joint wheel_front_drive_joint: origin xyz=0.0 -0.0482 -0.093 rpy=0 0 0 -> xyz=0.0 -0.0482 -0.0916 rpy=0 0 0
- joint wheel_front_left_joint: axis (none) -> 0 0 1; type fixed -> continuous
- joint wheel_front_right_joint: axis (none) -> 0 0 1; type fixed -> continuous
- joint wheel_rear_drive_joint: origin xyz=0.0 0.0482 -0.093 rpy=0 0 0 -> xyz=0.0 -0.0482 -0.0916 rpy=0 0 0
- joint wheel_rear_left_joint: axis (none) -> 0 0 1; type fixed -> continuous
- joint wheel_rear_right_joint: axis (none) -> 0 0 1; type fixed -> continuous

Commit message: Initial commit swerve_bringup

File: urdf/swerve_base.urdf (robot description, URDF)
Before this commit: robot agv_base, 13 links, 12 joints
Links:
- removed link wheel_front_left_link
- removed link wheel_front_right_link
- removed link wheel_rear_left_link
- removed link wheel_rear_right_link
Joints:
- removed joint wheel_front_left_joint
- removed joint wheel_front_right_joint
- removed joint wheel_rear_left_joint
- removed joint wheel_rear_right_joint

Commit message: m

File: urdf/swerve_base.urdf (robot description, URDF)
Before this commit: robot agv_base, 9 links, 8 joints
Links:
- link base_link: geometry collision box size=1.196 0.596 0.460; visual mesh filename=package://swerve_bringup/meshes/base_frame.stl scale=0.001 0.001 0.001
- link steer_front_link: geometry collision box size=0.2296 0.1862 0.2703; visual mesh filename=package://swerve_bringup/meshes/steer_front_housing_v2.stl scale=0.001 0.001 0.001
- link steer_rear_link: geometry collision box size=0.2296 0.1862 0.2834; visual mesh filename=package://swerve_bringup/meshes/steer_rear_housing_v2.stl scale=0.001 0.001 0.001
- link wheel_front_drive_link: geometry collision cylinder length=0.065 radius=0.0675; visual mesh filename=package://swerve_bringup/meshes/steer_front_wheel_v2.stl scale=0.001 0.001 0.001
- link wheel_rear_drive_link: geometry collision cylinder length=0.065 radius=0.0675; visual mesh filename=package://swerve_bringup/meshes/steer_rear_wheel_v2.stl scale=0.001 0.001 0.001

Commit message: feat: complete AGV visual model and runtime readiness

File: urdf/swerve_base.urdf (robot description, URDF)
Before this commit: robot agv_base, 9 links, 8 joints
Links:
- link base_link: geometry collision box size=1.196 0.596 0.460; visual box size=0.012 0.230 0.130
- link lidar_link: geometry collision cylinder length=0.07 radius=0.055; visual box size=0.020 0.012 0.006
- link steer_front_link: geometry collision box size=0.2296 0.1862 0.2703
- link steer_rear_link: geometry collision box size=0.2296 0.1862 0.2834
- link v30e_link: geometry visual box size=0.028 0.008 0.004; visual box size=0.09 0.07 0.025
- link wheel_front_drive_link: geometry collision cylinder length=0.065 radius=0.0675
- link wheel_rear_drive_link: geometry collision cylinder length=0.065 radius=0.0675
